Commit message: update vrx

File: wamv_gazebo/urdf/components/wamv_3d_lidar.xacro (robot description, xacro)
@@ -66,5 +66,5 @@
     <!-- Sensor post -->
     <link name="${namespace}/${name}_post_link">
-      <visual>
+      <!-- <visual>
         <geometry>
           <cylinder radius="${post_radius}" length="${post_length}"/>
@@ -73,5 +73,5 @@
           <color rgba="0.0 0.0 0.0 1.0"/>
         </material>
-      </visual>
+      </visual> -->
       <collision name="${name}_post_collision">
         <geometry>

File: wamv_gazebo/urdf/components/wamv_camera.xacro (robot description, xacro)
@@ -129,5 +129,5 @@
     <!-- Gazebo camera setup -->
     <gazebo reference="${namespace}/${name}_link">
-      <sensor type="camera" name="${name}_sensor">
+      <sensor type="depth" name="${name}_sensor">
         <update_rate>30.0</update_rate>
 	<xacro:if value="${visualize}">
@@ -135,9 +135,10 @@
 	</xacro:if>
         <camera name="${name}_camera">
-          <horizontal_fov>1.3962634</horizontal_fov>
+          <horizontal_fov>1.570796</horizontal_fov>
+          <vertical_fov>1.04872</vertical_fov>
           <image>
             <width>1280</width>
             <height>720</height>
-            <format>R8G8B8</format>
+            <format>B8G8R8</format>
           </image>
           <clip>
@@ -154,11 +155,17 @@
           </noise>
         </camera>
-        <plugin name="camera_plugin_${name}" filename="libgazebo_ros_camera.so">
+        <plugin name="camera_plugin_${name}" filename="libgazebo_ros_openni_kinect.so">
+          <baseline>0.2</baseline>
           <alwaysOn>true</alwaysOn>
-          <updateRate>0.0</updateRate>
+          <updateRate>1.0</updateRate>
           <cameraName>${namespace}/${sensor_namespace}${camera_namespace}${name}</cameraName>
           <imageTopicName>image_raw</imageTopicName>
           <cameraInfoTopicName>camera_info</cameraInfoTopicName>
+          <depthImageTopicName>depth/image_raw</depthImageTopicName>
+          <depthImageInfoTopicName>depth/camera_info</depthImageInfoTopicName>
+          <pointCloudTopicName>depth/points</pointCloudTopicName>
           <frameName>${namespace}/${name}_link_optical</frameName>
+          <pointCloudCutoff>0.5</pointCloudCutoff>
+          <pointCloudCutoffMax>25.0</pointCloudCutoffMax>
           <hackBaseline>0.07</hackBaseline>
           <distortionK1>0.0</distortionK1>
@@ -167,4 +174,9 @@
           <distortionT1>0.0</distortionT1>
           <distortionT2>0.0</distortionT2>
+          <CxPrime>0</CxPrime>
+          <Cx>0</Cx>
+          <Cy>0</Cy>
+          <focalLength>0</focalLength>
+          <hackBaseline>0</hackBaseline>
         </plugin>
       </sensor>

File: wamv_gazebo/urdf/thruster_layouts/wamv_t_thrusters_nycu.xacro (robot description, xacro)
@@ -4,6 +4,6 @@
   <xacro:engine prefix="left" position="-2.373776 1.027135 0.318237" />
   <xacro:engine prefix="right" position="-2.373776 -1.027135 0.318237" />
-  <xacro:engine prefix="left_lateral" position="1.33 0.90 0.318237" orientation="0.0 0.0 1.5707"/>
-  <xacro:engine prefix="right_lateral" position="1.33 -0.90 0.318237" orientation="0.0 0.0 -1.5707"/>
+  <xacro:engine prefix="left_lateral" position="1.20 0.90 0.318237" orientation="0.0 0.0 1.5707"/>
+  <xacro:engine prefix="right_lateral" position="1.20 -0.90 0.318237" orientation="0.0 0.0 -1.5707"/>
   <gazebo>
     <plugin name="wamv_gazebo_thrust" filename="libusv_gazebo_thrust_plugin.so">

File: wamv_gazebo/urdf/wamv_gazebo.urdf.xacro (robot description, xacro)
@@ -132,8 +132,8 @@
       <xacro:cpu_cases position="-0.15 0 1.53" orientation="0 0 0"/>
       <!-- Add a stereo camera pair -->
-      <!-- <xacro:wamv_camera name="front_left_camera" y="0.1" x="0.75" P="${radians(15)}" />
-      <xacro:wamv_camera name="front_right_camera" y="-0.1" x="0.75" P="${radians(15)}" /> -->
+      <xacro:wamv_camera name="left_camera" y="0.4" x="0.65" P="${radians(10)}" Y="${radians(30)}" post_Y="${radians(30)}"/>
+      <xacro:wamv_camera name="middle_camera" y="0" x="0.8" P="${radians(10)}" />
       <!-- Add a camera facing right -->
-      <xacro:wamv_camera name="middle_right_camera" y="-0.45" P="${radians(15)}" Y="${radians(-90)}" post_Y="${radians(-90)}" />
+      <xacro:wamv_camera name="right_camera" y="-0.4" x="0.65" P="${radians(10)}" Y="${radians(-30)}" post_Y="${radians(-30)}" />
       <!-- Add simulated GPS -->
       <xacro:wamv_gps name="gps_wamv" x="-0.85" />
@@ -141,9 +141,9 @@
       <xacro:wamv_imu name="imu_wamv" y="-0.2" />
       <!-- Add 3D LIDAR -->
-      <xacro:lidar name="lidar_wamv" type="16_beam"/>
+      <xacro:lidar name="lidar_wamv" x="1.25" y="0" z="1.0" type="16_beam"/>
       <!-- Add pinger -->
-      <xacro:wamv_pinger name="pinger" position="1.0 0 -1.0" />
+      <!-- <xacro:wamv_pinger name="pinger" position="1.0 0 -1.0" /> -->
       <!-- Add ball shooter (default pitch angle: ~-60 deg) -->
-      <xacro:wamv_ball_shooter name="ball_shooter" x="0.54" y="0.30" z="1.296" pitch="-1.04"/>
+      <!-- <xacro:wamv_ball_shooter name="ball_shooter" x="0.54" y="0.30" z="1.296" pitch="-1.04"/> -->
     </xacro:if>
   </xacro:unless>
