Commit message: narrow passage

File: vrx_gazebo/worlds/example_course_narrow.world.xacro (robot description, xacro)
@@ -21,9 +21,1164 @@
     <!-- The light buoy -->
     <include>
+      <uri>model://polyform_a7</uri>
+      <name>block00</name>
+      <pose>-600 -30 0 0 -0 0</pose>
+    </include>
+    <include>
+      <uri>model://polyform_a7</uri>
+      <name>block01</name>
+      <pose>-600 -32 0 0 -0 0</pose>
+    </include>
+    <include>
+      <uri>model://polyform_a7</uri>
+      <name>block02</name>
+      <pose>-600 -34 0 0 -0 0</pose>
+    </include>
+    <include>
+      <uri>model://polyform_a7</uri>
+      <name>block03</name>
+      <pose>-600 -36 0 0 -0 0</pose>
+    </include>
+    <include>
+      <uri>model://polyform_a7</uri>
+      <name>block04</name>
+      <pose>-600 -38 0 0 -0 0</pose>
+    </include>
+    <include>
+      <uri>model://polyform_a7</uri>
+      <name>block05</name>
+      <pose>-600 -40 0 0 -0 0</pose>
+    </include>
+    <include>
+      <uri>model://polyform_a7</uri>
+      <name>block06</name>
+      <pose>-600 -42 0 0 -0 0</pose>
+    </include>
+    <include>
+      <uri>model://polyform_a7</uri>
+      <name>block07</name>
+      <pose>-600 -44 0 0 -0 0</pose>
+    </include>
+    <include>
+      <uri>model://polyform_a7</uri>
+      <name>block08</name>
+      <pose>-600 -46 0 0 -0 0</pose>
+    </include>
+    <include>
+      <uri>model://polyform_a7</uri>
+      <name>block09</name>
+      <pose>-600 -48 0 0 -0 0</pose>
+    </include>
+    <include>
+      <uri>model://polyform_a7</uri>
+      <name>block10</name>
+      <pose>-600 -50 0 0 -0 0</pose>
+    </include>
+    <include>
+      <uri>model://polyform_a7</uri>
+      <name>block11</name>
+      <pose>-600 -52 0 0 -0 0</pose>
+    </include>
+    <include>
+      <uri>model://polyform_a7</uri>
+      <name>block12</name>
+      <pose>-600 -54 0 0 -0 0</pose>
+    </include>
+    <include>
+      <uri>model://polyform_a7</uri>
+      <name>block13</name>
+      <pose>-600 -56 0 0 -0 0</pose>
+    </include>
+    <include>
+      <uri>model://polyform_a7</uri>
+      <name>block14</name>
+      <pose>-600 -58 0 0 -0 0</pose>
+    </include>
+    <include>
+      <uri>model://polyform_a7</uri>
+      <name>block15</name>
+      <pose>-600 -60 0 0 -0 0</pose>
+    </include>
+    <include>
+      <uri>model://polyform_a7</uri>
+      <name>block16</name>
+      <pose>-600 -62 0 0 -0 0</pose>
+    </include>
+    <include>
+      <uri>model://polyform_a7</uri>
+      <name>block17</name>
+      <pose>-600 -64 0 0 -0 0</pose>
+    </include>
+    <include>
+      <uri>model://polyform_a7</uri>
+      <name>block18</name>
+      <pose>-600 -66 0 0 -0 0</pose>
+    </include>
+    <include>
+      <uri>model://polyform_a7</uri>
+      <name>block19</name>
+      <pose>-600 -68 0 0 -0 0</pose>
+    </include>
+    <include>
+      <uri>model://polyform_a7</uri>
+      <name>block20</name>
+      <pose>-600 -70 0 0 -0 0</pose>
+    </include>
+    <include>
+      <uri>model://polyform_a7</uri>
+      <name>block21</name>
+      <pose>-600 -72 0 0 -0 0</pose>
+    </include>
+    <include>
+      <uri>model://polyform_a7</uri>
+      <name>block22</name>
+      <pose>-600 -74 0 0 -0 0</pose>
+    </include>
+    <include>
+      <uri>model://polyform_a7</uri>
+      <name>block23</name>
+      <pose>-600 -76 0 0 -0 0</pose>
+    </include>
+    <include>
+      <uri>model://polyform_a7</uri>
+      <name>block24</name>
+      <pose>-600 -78 0 0 -0 0</pose>
+    </include>
+    <include>
+      <uri>model://polyform_a7</uri>
+      <name>block25</name>
+      <pose>-600 -80 0 0 -0 0</pose>
+    </include>
+    <include>
+      <uri>model://polyform_a7</uri>
+      <name>block26</name>
+      <pose>-600 -82 0 0 -0 0</pose>
+    </include>
+    <include>
+      <uri>model://polyform_a7</uri>
+      <name>block27</name>
+      <pose>-600 -84 0 0 -0 0</pose>
+    </include>
+    <include>
+      <uri>model://polyform_a7</uri>
+      <name>block28</name>
+      <pose>-600 -86 0 0 -0 0</pose>
+    </include>
+    <include>
+      <uri>model://polyform_a7</uri>
+      <name>block29</name>
+      <pose>-600 -88 0 0 -0 0</pose>
+    </include>
+    <include>
+      <uri>model://polyform_a7</uri>
+      <name>block30</name>
+      <pose>-600 -90 0 0 -0 0</pose>
+    </include>
+    <include>
+      <uri>model://polyform_a7</uri>
+      <name>block31</name>
+      <pose>-600 -92 0 0 -0 0</pose>
+    </include>
+    <include>
+      <uri>model://polyform_a7</uri>
+      <name>block32</name>
+      <pose>-600 -94 0 0 -0 0</pose>
+    </include>
+    <include>
+      <uri>model://polyform_a7</uri>
+      <name>block33</name>
+      <pose>-600 -94 0 0 -0 0</pose>
+    </include>
+    <include>
+      <uri>model://polyform_a7</uri>
+      <name>block34</name>
+      <pose>-600 -94 0 0 -0 0</pose>
+    </include>
+    <include>
+      <uri>model://polyform_a7</uri>
+      <name>block35</name>
+      <pose>-600 -94 0 0 -0 0</pose>
+    </include>
+    <include>
+      <uri>model://polyform_a7</uri>
+      <name>block36</name>
+      <pose>-600 -20 0 0 -0 0</pose>
+    </include>
+    <include>
+      <uri>model://polyform_a7</uri>
+      <name>block37</name>
+      <pose>-600 -18 0 0 -0 0</pose>
+    </include>
+    <include>
+      <uri>model://polyform_a7</uri>
+      <name>block38</name>
+      <pose>-600 -16 0 0 -0 0</pose>
+    </include>
+    <include>
+      <uri>model://polyform_a7</uri>
+      <name>block39</name>
+      <pose>-600 -14 0 0 -0 0</pose>
+    </include>
+    <include>
+      <uri>model://polyform_a7</uri>
+      <name>block40</name>
+      <pose>-600 -12 0 0 -0 0</pose>
+    </include>
+    <include>
+      <uri>model://polyform_a7</uri>
+      <name>block41</name>
+      <pose>-600 -10 0 0 -0 0</pose>
+    </include>
+    <include>
+      <uri>model://polyform_a7</uri>
+      <name>block42</name>
+      <pose>-600 -8 0 0 -0 0</pose>
+    </include>
+    <include>
+      <uri>model://polyform_a7</uri>
+      <name>block43</name>
+      <pose>-600 -6 0 0 -0 0</pose>
+    </include>
+    <include>
+      <uri>model://polyform_a7</uri>
+      <name>block44</name>
+      <pose>-600 -4 0 0 -0 0</pose>
+    </include>
+    <include>
+      <uri>model://polyform_a7</uri>
+      <name>block45</name>
+      <pose>-600 -2 0 0 -0 0</pose>
+    </include>
+    <include>
+      <uri>model://polyform_a7</uri>
+      <name>block46</name>
+      <pose>-600 0 0 0 -0 0</pose>
+    </include>
+    <include>
+      <uri>model://polyform_a7</uri>
+      <name>block47</name>
+      <pose>-600 2 0 0 -0 0</pose>
+    </include>
+    <include>
+      <uri>model://polyform_a7</uri>
+      <name>block48</name>
+      <pose>-600 4 0 0 -0 0</pose>
+    </include>
+    <include>
+      <uri>model://polyform_a7</uri>
+      <name>block49</name>
+      <pose>-600 6 0 0 -0 0</pose>
+    </include>
+    <include>
+      <uri>model://polyform_a7</uri>
+      <name>block50</name>
+      <pose>-600 8 0 0 -0 0</pose>
+    </include>
+    <include>
+      <uri>model://polyform_a7</uri>
+      <name>block51</name>
+      <pose>-600 10 0 0 -0 0</pose>
+    </include>
+    <include>
+      <uri>model://polyform_a7</uri>
+      <name>block52</name>
+      <pose>-600 12 0 0 -0 0</pose>
+    </include>
+    <include>
+      <uri>model://polyform_a7</uri>
+      <name>block53</name>
+      <pose>-600 14 0 0 -0 0</pose>
+    </include>
+    <include>
+      <uri>model://polyform_a7</uri>
+      <name>block54</name>
+      <pose>-600 16 0 0 -0 0</pose>
+    </include>
+    <include>
+      <uri>model://polyform_a7</uri>
+      <name>block55</name>
+      <pose>-600 18 0 0 -0 0</pose>
+    </include>
+    <include>
+      <uri>model://polyform_a7</uri>
+      <name>block56</name>
+      <pose>-600 20 0 0 -0 0</pose>
+    </include>
+    <include>
+      <uri>model://polyform_a7</uri>
+      <name>block57</name>
+      <pose>-600 22 0 0 -0 0</pose>
+    </include>
+    <include>
+      <uri>model://polyform_a7</uri>
+      <name>block58</name>
+      <pose>-600 24 0 0 -0 0</pose>
+    </include>
+    <include>
+      <uri>model://polyform_a7</uri>
+      <name>block59</name>
+      <pose>-600 26 0 0 -0 0</pose>
+    </include>
+    <include>
+      <uri>model://polyform_a7</uri>
+      <name>block60</name>
+      <pose>-600 28 0 0 -0 0</pose>
+    </include>
+    <include>
+      <uri>model://polyform_a7</uri>
+      <name>block61</name>
+      <pose>-600 30 0 0 -0 0</pose>
+    </include>
+    <include>
+      <uri>model://polyform_a7</uri>
+      <name>block62</name>
+      <pose>-600 32 0 0 -0 0</pose>
+    </include>
+    <include>
+      <uri>model://polyform_a7</uri>
+      <name>block63</name>
+      <pose>-600 34 0 0 -0 0</pose>
+    </include>
+    <include>
+      <uri>model://polyform_a7</uri>
+      <name>block64</name>
+      <pose>-600 36 0 0 -0 0</pose>
+    </include>
+    <include>
+      <uri>model://polyform_a7</uri>
+      <name>block65</name>
+      <pose>-600 38 0 0 -0 0</pose>
+    </include>
+    <include>
+      <uri>model://polyform_a7</uri>
+      <name>block66</name>
+      <pose>-600 40 0 0 -0 0</pose>
+    </include>
+    <include>
+      <uri>model://polyform_a7</uri>
+      <name>block67</name>
+      <pose>-600 42 0 0 -0 0</pose>
+    </include>
+    <include>
+      <uri>model://polyform_a7</uri>
+      <name>block68</name>
+      <pose>-600 44 0 0 -0 0</pose>
+    </include>
+    <include>
+      <uri>model://polyform_a7</uri>
+      <name>block69</name>
+      <pose>-600 46 0 0 -0 0</pose>
+    </include>
+    <include>
+      <uri>model://polyform_a7</uri>
+      <name>block70</name>
+      <pose>-600 48 0 0 -0 0</pose>
+    </include>
+    <include>
+      <uri>model://polyform_a7</uri>
+      <name>block71</name>
+      <pose>-600 50 0 0 -0 0</pose>
+    </include>
+    <include>
+      <uri>model://polyform_a7</uri>
+      <name>block72</name>
+      <pose>-600 52 0 0 -0 0</pose>
+    </include>
+    <include>
+      <uri>model://polyform_a7</uri>
+      <name>block73</name>
+      <pose>-600 54 0 0 -0 0</pose>
+    </include>
+    <include>
+      <uri>model://polyform_a7</uri>
+      <name>block74</name>
+      <pose>-600 56 0 0 -0 0</pose>
+    </include>
+    <include>
+      <uri>model://polyform_a7</uri>
+      <name>block75</name>
+      <pose>-600 58 0 0 -0 0</pose>
+    </include>
+    <include>
+      <uri>model://polyform_a7</uri>
+      <name>block76</name>
+      <pose>-600 60 0 0 -0 0</pose>
+    </include>
+    <include>
+      <uri>model://polyform_a7</uri>
+      <name>1block00</name>
+      <pose>-600 -30 0 0 -0 0</pose>
+    </include>
+    <include>
+      <uri>model://polyform_a7</uri>
+      <name>1block01</name>
+      <pose>-600 -32 0 0 -0 0</pose>
+    </include>
+    <include>
+      <uri>model://polyform_a7</uri>
+      <name>1block02</name>
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
File: wave_gazebo/world_models/ocean_waves/model.xacro (robot description, xacro)
@@ -17,5 +17,5 @@
 -->
 <world xmlns:xacro="http://ros.org/wiki/xacro">
-  <xacro:macro name="ocean_waves" params="gain:=0.1 period:=5
+  <xacro:macro name="ocean_waves" params="gain:=1 period:=2
                      direction_x:=1.0 direction_y:=0.0
                      angle:=0.4 scale:=1.5">

Commit message: 1 row environment

File: vrx_gazebo/worlds/example_course_narrow.world.xacro (robot description, xacro)
@@ -405,4 +405,5 @@
       <pose>-600 60 0 0 -0 0</pose>
     </include>
+<!--
     <include>
       <uri>model://polyform_a7</uri>
@@ -1175,4 +1176,5 @@
       <pose>-600 60 0 0 -0 0</pose>
     </include>
+ -->
     <include>
       <uri>model://robotx_light_buoy</uri>

File: wave_gazebo/world_models/ocean_waves/model.xacro (robot description, xacro)
@@ -17,5 +17,5 @@
 -->
 <world xmlns:xacro="http://ros.org/wiki/xacro">
-  <xacro:macro name="ocean_waves" params="gain:=1 period:=2
+  <xacro:macro name="ocean_waves" params="gain:=0.1 period:=5
                      direction_x:=1.0 direction_y:=0.0
                      angle:=0.4 scale:=1.5">
