Commit message: add record.sh change large wave

File: wave_gazebo/world_models/ocean_waves/model.xacro (robot description, xacro)
@@ -17,5 +17,5 @@
 -->
 <world xmlns:xacro="http://ros.org/wiki/xacro">
-  <xacro:macro name="ocean_waves" params="gain:=0.1 period:=5
+  <xacro:macro name="ocean_waves" params="gain:=1 period:=3
                      direction_x:=1.0 direction_y:=0.0
                      angle:=0.4 scale:=1.5">

Commit message: add motor anchor world

File: wave_gazebo/world_models/ocean_waves/model.xacro (robot description, xacro)
@@ -17,5 +17,5 @@
 -->
 <world xmlns:xacro="http://ros.org/wiki/xacro">
-  <xacro:macro name="ocean_waves" params="gain:=1 period:=3
+  <xacro:macro name="ocean_waves" params="gain:=0.1 period:=5
                      direction_x:=1.0 direction_y:=0.0
                      angle:=0.4 scale:=1.5">
