Commit message: Feat: Add Mavlink into wamv

File: wamv_gazebo/urdf/macros.xacro (robot description, xacro)
@@ -14,4 +14,5 @@
   <xacro:include filename="$(find wamv_gazebo)/urdf/components/wamv_p3d.xacro" />
   <xacro:include filename="$(find wamv_gazebo)/urdf/components/wamv_pinger.xacro" />
+  <xacro:include filename="$(find wamv_gazebo)/urdf/components/wamv_mavlink.xacro"/>
   <!-- Include ball shooter macros -->
   <xacro:include filename="$(find wamv_gazebo)/urdf/components/ball_shooter.xacro" />

File: wamv_gazebo/urdf/wamv_gazebo.urdf.xacro (robot description, xacro)
@@ -1,6 +1,5 @@
 <?xml version="1.0"?>
 <!-- Basic WAM-V with gazebo plugins for dynamics -->
-<robot xmlns:xacro="http://ros.org/wiki/xacro"
-       name="WAM-V">
+<robot xmlns:xacro="http://ros.org/wiki/xacro" name="WAM-V">
   <xacro:arg name="locked" default="false" />
   <xacro:arg name="thruster_config" default="" />
@@ -34,4 +33,5 @@
   <xacro:arg name="thruster_xacro_file" default = ""/>
   <xacro:arg name="plate" default="false" />
+  <xacro:arg name="mavlink_enabled" default="false" />
   <!-- === The WAM-V platform === -->
   <xacro:include filename="$(find wamv_gazebo)/urdf/wamv_gazebo.xacro"/>
@@ -50,5 +50,5 @@
     <!-- Default WAM-V with two aft thrusters -->
     <xacro:if value="${thruster_conf == 'H'}">
-       <xacro:wamv_gazebo thruster_layout="$(find wamv_gazebo)/urdf/thruster_layouts/wamv_aft_thrusters.xacro"/>
+      <xacro:wamv_gazebo thruster_layout="$(find wamv_gazebo)/urdf/thruster_layouts/wamv_aft_thrusters.xacro"/>
     </xacro:if>
     <!-- WAMV with "T" thruster configuration -->
@@ -155,23 +155,26 @@
       <!-- Add ball shooter (default pitch angle: ~-60 deg) -->
       <!-- <xacro:wamv_ball_shooter name="ball_shooter" x="0.54" y="0.30" z="1.296" pitch="-1.04"/> -->
-      <xacro:if value="$(arg plate)">
-        <link name="$(arg namespace)/plate">
-          <visual>
-            <geometry>
-              <box size="1.5 1.0 0.01"/>
-            </geometry>
-          </visual>
-          <collision>
-            <geometry>
-              <box size="1.5 1.0 0.01"/>
-            </geometry>
-          </collision>
-        </link>
-        <joint name="base_to_plate" type="fixed">
-          <parent link="$(arg namespace)/base_link"/>
-          <child link="$(arg namespace)/plate"/>
-          <origin xyz="0 0 1.85"/>
-        </joint>
-      </xacro:if>
+    </xacro:if>
+    <xacro:if value="$(arg plate)">
+      <link name="$(arg namespace)/plate">
+        <visual>
+          <geometry>
+            <box size="1.5 1.0 0.01"/>
+          </geometry>
+        </visual>
+        <collision>
+          <geometry>
+            <box size="1.5 1.0 0.01"/>
+          </geometry>
+        </collision>
+      </link>
+      <joint name="base_to_plate" type="fixed">
+        <parent link="$(arg namespace)/base_link"/>
+        <child link="$(arg namespace)/plate"/>
+        <origin xyz="0 0 1.85"/>
+      </joint>
+    </xacro:if>
+    <xacro:if value="$(arg mavlink_enabled)">
+      <xacro:wamv_mavlink name="mavlink_wamv"/>
     </xacro:if>
   </xacro:unless>
