Commit message: Feat: Add top plate for UAV landing

File: wamv_gazebo/urdf/wamv_gazebo.urdf.xacro (robot description, xacro)
@@ -4,5 +4,5 @@
        name="WAM-V">
   <xacro:arg name="locked" default="false" />
-  <xacro:arg name="thruster_config" default="H" />
+  <xacro:arg name="thruster_config" default="" />
   <xacro:arg name="camera_enabled" default="false" />
   <xacro:arg name="gps_enabled" default="false" />
@@ -33,4 +33,5 @@
   <xacro:arg name="yaml_thruster_generation" default="false"/>
   <xacro:arg name="thruster_xacro_file" default = ""/>
+  <xacro:arg name="plate" default="false" />
   <!-- === The WAM-V platform === -->
   <xacro:include filename="$(find wamv_gazebo)/urdf/wamv_gazebo.xacro"/>
@@ -58,4 +59,8 @@
     <xacro:if value="${thruster_conf == 'X'}">
       <xacro:wamv_gazebo thruster_layout="$(find wamv_gazebo)/urdf/thruster_layouts/wamv_x_thrusters.xacro"/>
+    </xacro:if>
+    <!-- WAMV with "X" thruster configuration -->
+    <xacro:if value="${thruster_conf == ''}">
+      <xacro:wamv_gazebo thruster_layout=""/>
     </xacro:if>
   </xacro:unless>
@@ -146,4 +151,23 @@
       <!-- Add ball shooter (default pitch angle: ~-60 deg) -->
       <!-- <xacro:wamv_ball_shooter name="ball_shooter" x="0.54" y="0.30" z="1.296" pitch="-1.04"/> -->
+      <xacro:if value="$(arg plate)">
+        <link name="$(arg namespace)/plate">
+          <visual>
+            <geometry>
+              <box size="3.0 3.0 0.01"/>
+            </geometry>
+          </visual>
+          <collision>
+            <geometry>
+              <box size="3.0 3.0 0.01"/>
+            </geometry>
+          </collision>
+        </link>
+        <joint name="base_to_plate" type="fixed">
+          <parent link="$(arg namespace)/base_link"/>
+          <child link="$(arg namespace)/plate"/>
+          <origin xyz="0 0 1.85"/>
+        </joint>
+      </xacro:if>
     </xacro:if>
   </xacro:unless>

File: wamv_gazebo/urdf/wamv_gazebo.xacro (robot description, xacro)
@@ -8,5 +8,7 @@
     <xacro:include filename="$(find wamv_description)/urdf/wamv_base_contact.urdf.xacro" />
     <!-- Thruster Layout -->
-    <xacro:include filename="${thruster_layout}"/>
+    <xacro:if value="${thruster_layout != ''}">
+      <xacro:include filename="${thruster_layout}"/>
+    </xacro:if>
     <!-- Attach hydrodynamics plugin -->
     <xacro:usv_dynamics_gazebo name="wamv_dynamics_plugin"/>

Commit message: Feat: Add drone with uwb launch

File: wamv_gazebo/urdf/wamv_gazebo.urdf.xacro (robot description, xacro)
@@ -159,10 +159,10 @@
           <visual>
             <geometry>
-              <box size="3.0 3.0 0.01"/>
+              <box size="1.5 1.0 0.01"/>
             </geometry>
           </visual>
           <collision>
             <geometry>
-              <box size="3.0 3.0 0.01"/>
+              <box size="1.5 1.0 0.01"/>
             </geometry>
           </collision>

Commit message: Feat: Add red ball to wamv

File: wamv_gazebo/urdf/wamv_gazebo.urdf.xacro (robot description, xacro)
@@ -34,4 +34,5 @@
   <xacro:arg name="plate" default="false" />
   <xacro:arg name="mavlink_enabled" default="false" />
+  <xacro:arg name="red_ball" default="false" />
   <!-- === The WAM-V platform === -->
   <xacro:include filename="$(find wamv_gazebo)/urdf/wamv_gazebo.xacro"/>
@@ -178,4 +179,26 @@
       <xacro:wamv_mavlink name="mavlink_wamv"/>
     </xacro:if>
+    <xacro:if value="$(arg red_ball)">
+      <link name="$(arg namespace)/red_ball">
+        <visual>
+          <geometry>
+            <sphere radius="0.1"/>
+          </geometry>
+        </visual>
+        <collision>
+          <geometry>
+            <sphere radius="0.1"/>
+          </geometry>
+        </collision>
+      </link>
+      <joint name="base_to_red_ball" type="fixed">
+        <parent link="$(arg namespace)/base_link"/>
+        <child link="$(arg namespace)/red_ball"/>
+        <origin xyz="-0.2 0 1.8"/>
+      </joint>
+      <gazebo reference="${namespace}/red_ball">
+        <material>Gazebo/Red</material>
+      </gazebo>
+    </xacro:if>
   </xacro:unless>
 </robot>

Commit message: Feat: Add red torus into wamv

File: wamv_gazebo/urdf/wamv_gazebo.urdf.xacro (robot description, xacro)
@@ -12,12 +12,12 @@
   <xacro:arg name="pinger_enabled" default="false" />
   <xacro:arg name="ball_shooter_enabled" default="false" />
-  <xacro:arg name="thruster_namespace" default="thrusters/"/>
-  <xacro:arg name="camera_namespace" default="cameras/"/>
-  <xacro:arg name="sensor_namespace" default="sensors/"/>
-  <xacro:arg name="pinger_namespace" default="pingers/"/>
-  <xacro:arg name="shooter_namespace" default="shooters/"/>
+  <xacro:arg name="thruster_namespace" default="thrusters/" />
+  <xacro:arg name="camera_namespace" default="cameras/" />
+  <xacro:arg name="sensor_namespace" default="sensors/" />
+  <xacro:arg name="pinger_namespace" default="pingers/" />
+  <xacro:arg name="shooter_namespace" default="shooters/" />
   <!-- Note: this is only used for some sensors that do not correctly use the
   robotNamespace parameter -->
-  <xacro:arg name="namespace" default="wamv"/>
+  <xacro:arg name="namespace" default="wamv" />
   <xacro:property name="thruster_namespace" value="$(arg thruster_namespace)" scope="global" />
   <xacro:property name="camera_namespace" value="$(arg camera_namespace)" scope="global" />
@@ -27,45 +27,50 @@
   <xacro:property name="namespace" value="$(arg namespace)" scope="global" />
   <!-- Sensor yaml file -->
-  <xacro:arg name="yaml_component_generation" default="false"/>
-  <xacro:arg name="component_xacro_file" default = ""/>
+  <xacro:arg name="yaml_component_generation" default="false" />
+  <xacro:arg name="component_xacro_file" default="" />
   <!-- Thruster yaml file -->
-  <xacro:arg name="yaml_thruster_generation" default="false"/>
-  <xacro:arg name="thruster_xacro_file" default = ""/>
+  <xacro:arg name="yaml_thruster_generation" default="false" />
+  <xacro:arg name="thruster_xacro_file" default="" />
   <xacro:arg name="plate" default="false" />
   <xacro:arg name="mavlink_enabled" default="false" />
   <xacro:arg name="red_ball" default="false" />
+  <xacro:arg name="red_torus" default="false" />
   <!-- === The WAM-V platform === -->
-  <xacro:include filename="$(find wamv_gazebo)/urdf/wamv_gazebo.xacro"/>
+  <xacro:include filename="$(find wamv_gazebo)/urdf/wamv_gazebo.xacro" />
   <!-- === Batteries === -->
-  <xacro:include filename="$(find wamv_description)/urdf/battery.xacro"/>
-  <xacro:battery prefix="left" position="0 1 0.45" orientation="0 0 0"/>
-  <xacro:battery prefix="right" position="0 -1 0.45" orientation="0 0 0"/>
+  <xacro:include filename="$(find wamv_description)/urdf/battery.xacro" />
+  <xacro:battery prefix="left" position="0 1 0.45" orientation="0 0 0" />
+  <xacro:battery prefix="right" position="0 -1 0.45" orientation="0 0 0" />
   <!-- === Thrusters === -->
   <!-- Use thruster yaml file if given -->
   <xacro:if value="$(arg yaml_thruster_generation)">
-    <xacro:wamv_gazebo thruster_layout="$(arg thruster_xacro_file)"/>
+    <xacro:wamv_gazebo thruster_layout="$(arg thruster_xacro_file)" />
   </xacro:if>
   <!-- Otherwise, add thrusters based on thruster_config variable -->
   <xacro:unless value="$(arg yaml_thruster_generation)">
-    <xacro:property name="thruster_conf" value="$(arg thruster_config)"/>
+    <xacro:property name="thruster_conf" value="$(arg thruster_config)" />
     <!-- Default WAM-V with two aft thrusters -->
     <xacro:if value="${thruster_conf == 'H'}">
-      <xacro:wamv_gazebo thruster_layout="$(find wamv_gazebo)/urdf/thruster_layouts/wamv_aft_thrusters.xacro"/>
+      <xacro:wamv_gazebo
+        thruster_layout="$(find wamv_gazebo)/urdf/thruster_layouts/wamv_aft_thrusters.xacro" />
     </xacro:if>
     <!-- WAMV with "T" thruster configuration -->
     <xacro:if value="${thruster_conf == 'T'}">
-      <xacro:wamv_gazebo thruster_layout="$(find wamv_gazebo)/urdf/thruster_layouts/wamv_t_thrusters_nycu.xacro"/>
+      <xacro:wamv_gazebo
+        thruster_layout="$(find wamv_gazebo)/urdf/thruster_layouts/wamv_t_thrusters_nycu.xacro" />
     </xacro:if>
     <!-- WAMV with "X" thruster configuration -->
     <xacro:if value="${thruster_conf == 'X'}">
-      <xacro:wamv_gazebo thruster_layout="$(find wamv_gazebo)/urdf/thruster_layouts/wamv_x_thrusters.xacro"/>
+      <xacro:wamv_gazebo
+        thruster_layout="$(find wamv_gazebo)/urdf/thruster_layouts/wamv_x_thrusters.xacro" />
     </xacro:if>
     <!-- WAMV with "X_square" thruster configuration -->
     <xacro:if value="${thruster_conf == 'X_square'}">
-      <xacro:wamv_gazebo thruster_layout="$(find wamv_gazebo)/urdf/thruster_layouts/wamv_x_square_thrusters.xacro"/>
+      <xacro:wamv_gazebo
+        thruster_layout="$(find wamv_gazebo)/urdf/thruster_layouts/wamv_x_square_thrusters.xacro" />
     </xacro:if>
     <!-- WAMV with "X" thruster configuration -->
     <xacro:if value="${thruster_conf == ''}">
-      <xacro:wamv_gazebo thruster_layout=""/>
+      <xacro:wamv_gazebo thruster_layout="" />
     </xacro:if>
   </xacro:unless>
@@ -73,5 +78,5 @@
   <xacro:if value="$(arg locked)">
     <gazebo>
-      <link name="wamv_external_link"/>
+      <link name="wamv_external_link" />
       <joint name="wamv_external_pivot_joint" type="universal">
         <parent>wamv::wamv/base_link</parent>
@@ -100,9 +105,9 @@
   <!-- Use sensor yaml file if given -->
   <xacro:if value="$(arg yaml_component_generation)">
-    <xacro:include filename="$(arg component_xacro_file)"/>
+    <xacro:include filename="$(arg component_xacro_file)" />
     <xacro:yaml_components />
     <!-- Add CPU Cases -->
     <xacro:include filename="$(find wamv_description)/urdf/cpu_cases.xacro" />
-    <xacro:cpu_cases position="-0.15 0 1.53" orientation="0 0 0"/>
+    <xacro:cpu_cases position="-0.15 0 1.53" orientation="0 0 0" />
   </xacro:if>
   <!-- Otherwise, add sensors based on enable variables -->
@@ -122,9 +127,9 @@
     <!-- Add 3D LIDAR -->
     <xacro:if value="$(arg lidar_enabled)">
-      <xacro:lidar name="lidar_wamv" y="-0.3" type="16_beam"/>
+      <xacro:lidar name="lidar_wamv" y="-0.3" type="16_beam" />
     </xacro:if>
     <!-- Add P3D ground truth -->
     <xacro:if value="$(arg ground_truth_enabled)">
-      <xacro:wamv_p3d name="p3d_wamv"/>
+      <xacro:wamv_p3d name="p3d_wamv" />
     </xacro:if>
     <!-- Add pinger -->
@@ -134,5 +139,5 @@
     <!-- Add ball shooter (default pitch angle: ~-60 deg) -->
     <xacro:if value="$(arg ball_shooter_enabled)">
-      <xacro:wamv_ball_shooter name="ball_shooter" x="0.54" y="0.30" z="1.296" pitch="-1.04"/>
+      <xacro:wamv_ball_shooter name="ball_shooter" x="0.54" y="0.30" z="1.296" pitch="-1.04" />
     </xacro:if>
     <!-- ==== VRX sensor configuration ==== -->
@@ -140,10 +145,12 @@
       <!-- Add CPU Cases -->
       <xacro:include filename="$(find wamv_description)/urdf/cpu_cases.xacro" />
-      <xacro:cpu_cases position="-0.15 0 1.53" orientation="0 0 0"/>
+      <xacro:cpu_cases position="-0.15 0 1.53" orientation="0 0 0" />
       <!-- Add a stereo camera pair -->
-      <xacro:wamv_camera name="left_camera" y="0.4" x="0.65" P="${radians(10)}" Y="${radians(30)}" post_Y="${radians(30)}"/>
+      <xacro:wamv_camera name="left_camera" y="0.4" x="0.65" P="${radians(10)}" Y="${radians(30)}"
+        post_Y="${radians(30)}" />
       <xacro:wamv_camera name="middle_camera" y="0" x="0.8" P="${radians(10)}" />
       <!-- Add a camera facing right -->
-      <xacro:wamv_camera name="right_camera" y="-0.4" x="0.65" P="${radians(10)}" Y="${radians(-30)}" post_Y="${radians(-30)}" />
+      <xacro:wamv_camera name="right_camera" y="-0.4" x="0.65" P="${radians(10)}"
+        Y="${radians(-30)}" post_Y="${radians(-30)}" />
       <!-- Add simulated GPS -->
       <xacro:wamv_gps name="gps_wamv" x="-0.85" />
@@ -151,5 +158,5 @@
       <xacro:wamv_imu name="imu_wamv" y="-0.2" />
       <!-- Add 3D LIDAR -->
-      <xacro:lidar name="lidar_wamv" x="1.45" y="0" z="1.0" type="16_beam"/>
+      <xacro:lidar name="lidar_wamv" x="1.45" y="0" z="1.0" type="16_beam" />
       <!-- Add pinger -->
       <!-- <xacro:wamv_pinger name="pinger" position="1.0 0 -1.0" /> -->
@@ -161,21 +168,21 @@
         <visual>
           <geometry>
-            <box size="1.5 1.0 0.01"/>
+            <box size="1.5 1.0 0.01" />
           </geometry>
         </visual>
         <collision>
           <geometry>
-            <box size="1.5 1.0 0.01"/>
+            <box size="1.5 1.0 0.01" />
           </geometry>
         </collision>
       </link>
       <joint name="base_to_plate" type="fixed">
-        <parent link="$(arg namespace)/base_link"/>
-        <child link="$(arg namespace)/plate"/>
-        <origin xyz="0 0 1.85"/>
+        <parent link="$(arg namespace)/base_link" />
+        <child link="$(arg namespace)/plate" />
+        <origin xyz="0 0 1.85" />
       </joint>
     </xacro:if>
     <xacro:if value="$(arg mavlink_enabled)">
-      <xacro:wamv_mavlink name="mavlink_wamv"/>
+      <xacro:wamv_mavlink name="mavlink_wamv" />
     </xacro:if>
     <xacro:if value="$(arg red_ball)">
@@ -183,17 +190,17 @@
         <visual>
           <geometry>
-            <sphere radius="0.1"/>
+            <sphere radius="0.1" />
           </geometry>
         </visual>
         <collision>
           <geometry>
-            <sphere radius="0.1"/>
+            <sphere radius="0.1" />
           </geometry>
         </collision>
       </link>
-      <joint name="base_to_red_ball" type="fixed">
-        <parent link="$(arg namespace)/base_link"/>
-        <child link="$(arg namespace)/red_ball"/>
-        <origin xyz="-0.2 0 1.8"/>
+      <joint name="red_ball_joint" type="fixed">
+        <parent link="$(arg namespace)/base_link" />
+        <child link="$(arg namespace)/red_ball" />
+        <origin xyz="-0.2 0 1.9" />
       </joint>
       <gazebo reference="${namespace}/red_ball">
@@ -201,4 +208,30 @@
       </gazebo>
     </xacro:if>
+    <xacro:if value="$(arg red_torus)">
+      <material name="Red">
+        <color rgba="1.0 0.0 0.0 1.0"/>
+      </material>
+      <link name="$(arg namespace)/red_torus_link">
+        <visual>
+          <geometry>
+            <mesh filename="package://wamv_description/models/torus.stl" />
+          </geometry>
+          <material name="Red"/>
+        </visual>
+        <collision>
+          <geometry>
+            <mesh filename="package://wamv_description/models/torus.stl" />
+          </geometry>
+        </collision>
+      </link>
+      <joint name="red_torus_joint" type="fixed">
+        <parent link="$(arg namespace)/base_link" />
+        <child link="$(arg namespace)/red_torus_link" />
+        <origin xyz="-0.2 0 2.2" />
+      </joint>
+      <gazebo reference="$(arg namespace)/red_torus_link">
+        <material>Gazebo/Red</material>
+      </gazebo>
+    </xacro:if>
   </xacro:unless>
 </robot>

Commit message: Fix: Move top plate colision center

File: wamv_gazebo/urdf/wamv_gazebo.urdf.xacro (robot description, xacro)
@@ -180,5 +180,5 @@
         <parent link="$(arg namespace)/base_link" />
         <child link="$(arg namespace)/plate" />
-        <origin xyz="0 0 1.85" />
+        <origin xyz="-0.24 0 1.78" />
       </joint>
     </xacro:if>

Commit message: Update wamv and drone

File: wamv_gazebo/urdf/wamv_gazebo.urdf.xacro (robot description, xacro)
@@ -32,5 +32,6 @@
   <xacro:arg name="yaml_thruster_generation" default="false" />
   <xacro:arg name="thruster_xacro_file" default="" />
-  <xacro:arg name="plate" default="false" />
+  <xacro:arg name="helipad_plate" default="false" />
+  <xacro:arg name="holed_helipad_plate" default="false" />
   <xacro:arg name="mavlink_enabled" default="false" />
   <xacro:arg name="red_ball" default="false" />
@@ -52,21 +53,17 @@
     <!-- Default WAM-V with two aft thrusters -->
     <xacro:if value="${thruster_conf == 'H'}">
-      <xacro:wamv_gazebo
-        thruster_layout="$(find wamv_gazebo)/urdf/thruster_layouts/wamv_aft_thrusters.xacro" />
+      <xacro:wamv_gazebo thruster_layout="$(find wamv_gazebo)/urdf/thruster_layouts/wamv_aft_thrusters.xacro" />
     </xacro:if>
     <!-- WAMV with "T" thruster configuration -->
     <xacro:if value="${thruster_conf == 'T'}">
-      <xacro:wamv_gazebo
-        thruster_layout="$(find wamv_gazebo)/urdf/thruster_layouts/wamv_t_thrusters_nycu.xacro" />
+      <xacro:wamv_gazebo thruster_layout="$(find wamv_gazebo)/urdf/thruster_layouts/wamv_t_thrusters_nycu.xacro" />
     </xacro:if>
     <!-- WAMV with "X" thruster configuration -->
     <xacro:if value="${thruster_conf == 'X'}">
-      <xacro:wamv_gazebo
-        thruster_layout="$(find wamv_gazebo)/urdf/thruster_layouts/wamv_x_thrusters.xacro" />
+      <xacro:wamv_gazebo thruster_layout="$(find wamv_gazebo)/urdf/thruster_layouts/wamv_x_thrusters.xacro" />
     </xacro:if>
     <!-- WAMV with "X_square" thruster configuration -->
     <xacro:if value="${thruster_conf == 'X_square'}">
-      <xacro:wamv_gazebo
-        thruster_layout="$(find wamv_gazebo)/urdf/thruster_layouts/wamv_x_square_thrusters.xacro" />
+      <xacro:wamv_gazebo thruster_layout="$(find wamv_gazebo)/urdf/thruster_layouts/wamv_x_square_thrusters.xacro" />
     </xacro:if>
     <!-- WAMV with "X" thruster configuration -->
@@ -147,10 +144,8 @@
       <xacro:cpu_cases position="-0.15 0 1.53" orientation="0 0 0" />
       <!-- Add a stereo camera pair -->
-      <xacro:wamv_camera name="left_camera" y="0.4" x="0.65" P="${radians(10)}" Y="${radians(30)}"
-        post_Y="${radians(30)}" />
+      <xacro:wamv_camera name="left_camera" y="0.4" x="0.65" P="${radians(10)}" Y="${radians(30)}" post_Y="${radians(30)}" />
       <xacro:wamv_camera name="middle_camera" y="0" x="0.8" P="${radians(10)}" />
       <!-- Add a camera facing right -->
-      <xacro:wamv_camera name="right_camera" y="-0.4" x="0.65" P="${radians(10)}"
-        Y="${radians(-30)}" post_Y="${radians(-30)}" />
+      <xacro:wamv_camera name="right_camera" y="-0.4" x="0.65" P="${radians(10)}" Y="${radians(-30)}" post_Y="${radians(-30)}" />
       <!-- Add simulated GPS -->
       <xacro:wamv_gps name="gps_wamv" x="-0.85" />
@@ -164,20 +159,55 @@
       <!-- <xacro:wamv_ball_shooter name="ball_shooter" x="0.54" y="0.30" z="1.296" pitch="-1.04"/> -->
     </xacro:if>
-    <xacro:if value="$(arg plate)">
-      <link name="$(arg namespace)/plate">
-        <visual>
-          <geometry>
+    <xacro:if value="$(arg helipad_plate)">
+      <link name="$(arg namespace)/helipad_plate">
+        <visual>
+          <geometry>
+            <!-- <mesh filename="package://wamv_description/models/helipad.dae" /> -->
             <box size="1.5 1.0 0.01" />
           </geometry>
         </visual>
-        <collision>
-          <geometry>
+        <collision name="helipad_plate_collision">
+          <geometry>
+            <!-- <mesh filename="package://wamv_description/models/helipad.dae" /> -->
             <box size="1.5 1.0 0.01" />
           </geometry>
         </collision>
-      </link>
-      <joint name="base_to_plate" type="fixed">
-        <parent link="$(arg namespace)/base_link" />
-        <child link="$(arg namespace)/plate" />
+        <collision name="cylinder_collision">
+          <origin xyz="0 0 0" rpy="0 0 0"/>
+          <geometry>
+            <cylinder radius="0.1" length="0.01"/>
+          </geometry>
+        </collision>
+      </link>
+      <joint name="base_to_helipad_plate" type="fixed">
+        <parent link="$(arg namespace)/base_link" />
+        <child link="$(arg namespace)/helipad_plate" />
+        <origin xyz="-0.24 0 1.77" />
+      </joint>
+    </xacro:if>
+    <xacro:if value="$(arg holed_helipad_plate)">
+      <link name="$(arg namespace)/holed_helipad_plate">
+        <visual>
+          <geometry>
+            <mesh filename="package://wamv_description/models/helipad_hole.dae" />
+            <!-- <box size="1.5 1.0 0.01" /> -->
+          </geometry>
+        </visual>
+        <collision name="helipad_plate_collision">
+          <geometry>
+            <mesh filename="package://wamv_description/models/helipad_hole.dae" />
+            <!-- <box size="1.5 1.0 0.01" /> -->
+          </geometry>
+        </collision>
+        <collision name="cylinder_collision">
+          <origin xyz="0 0 0" rpy="0 0 0"/>
+          <geometry>
+            <cylinder radius="0.1" length="0.01"/>
+          </geometry>
+        </collision>
+      </link>
+      <joint name="base_to_holed_helipad_plate" type="fixed">
+        <parent link="$(arg namespace)/base_link" />
+        <child link="$(arg namespace)/holed_helipad_plate" />
         <origin xyz="-0.24 0 1.78" />
       </joint>

Commit message: Update wamv torous height

File: wamv_gazebo/urdf/wamv_gazebo.urdf.xacro (robot description, xacro)
@@ -258,5 +258,5 @@
         <parent link="$(arg namespace)/base_link" />
         <child link="$(arg namespace)/red_torus_link" />
-        <origin xyz="-0.2 0 2.2" />
+        <origin xyz="-0.2 0 2" />
       </joint>
       <gazebo reference="$(arg namespace)/red_torus_link">

Commit message: Update wamv_gazebo.urdf.xacro

File: wamv_gazebo/urdf/wamv_gazebo.urdf.xacro (robot description, xacro)
@@ -37,4 +37,5 @@
   <xacro:arg name="red_ball" default="false" />
   <xacro:arg name="red_torus" default="false" />
+  <xacro:arg name="green_landing_cylinder" default="true" />
   <!-- === The WAM-V platform === -->
   <xacro:include filename="$(find wamv_gazebo)/urdf/wamv_gazebo.xacro" />
@@ -264,4 +265,27 @@
       </gazebo>
     </xacro:if>
+    <xacro:if value="$(arg green_landing_cylinder)">
+      <link name="$(arg namespace)/green_landing_cylinder_link">
+        <visual>
+          <geometry>
+            <cylinder radius="0.1" length="0.01"/>
+          </geometry>
+          <material name="Green"/>
+        </visual>
+        <collision>
+          <geometry>
+            <cylinder radius="0.1" length="0.01"/>
+          </geometry>
+        </collision>
+      </link>
+      <joint name="green_landing_cylinder_joint" type="fixed">
+        <parent link="$(arg namespace)/base_link" />
+        <child link="$(arg namespace)/green_landing_cylinder_link" />
+        <origin xyz="-0.24 0 1.78" />
+      </joint>
+      <gazebo reference="$(arg namespace)/green_landing_cylinder_link">
+        <material>Gazebo/Green</material>
+      </gazebo>
+    </xacro:if>
   </xacro:unless>
 </robot>
