Commit message: fix contact sensor

File: wamv_description/urdf/wamv_base_contact.urdf.xacro (robot description, xacro)
@@ -91,10 +91,10 @@
             <updaterate>100.0</updaterate>
             <contact>
-                <collision>${namespace}/base_link_fixed_joint_lump__left_float_collision_9</collision>
-                <collision>${namespace}/base_link_fixed_joint_lump__left_mid_float_collision_10</collision>
-                <collision>${namespace}/base_link_fixed_joint_lump__left_front_float_collision_11</collision>
-                <collision>${namespace}/base_link_fixed_joint_lump__right_float_collision_21</collision>
-                <collision>${namespace}/base_link_fixed_joint_lump__right_mid_float_collision_22</collision>
-                <collision>${namespace}/base_link_fixed_joint_lump__right_front_float_collision_23</collision>
+                <collision>${namespace}/base_link_fixed_joint_lump__left_float_collision_17</collision>
+                <collision>${namespace}/base_link_fixed_joint_lump__left_mid_float_collision_18</collision>
+                <collision>${namespace}/base_link_fixed_joint_lump__left_front_float_collision_19</collision>
+                <collision>${namespace}/base_link_fixed_joint_lump__right_float_collision_29</collision>
+                <collision>${namespace}/base_link_fixed_joint_lump__right_mid_float_collision_30</collision>
+                <collision>${namespace}/base_link_fixed_joint_lump__right_front_float_collision_31</collision>
             </contact>
             <plugin name="gazebo_ros_bumper_controller" filename="libgazebo_ros_bumper.so">

File: wamv_gazebo/urdf/wamv_gazebo.xacro (robot description, xacro)
@@ -6,5 +6,5 @@
   <xacro:macro  name="wamv_gazebo" params="thruster_layout">
     <!-- Defines the base vehicle -->
-    <xacro:include filename="$(find wamv_description)/urdf/wamv_base.urdf.xacro" />
+    <xacro:include filename="$(find wamv_description)/urdf/wamv_base_contact_old.urdf.xacro" />
     <!-- Thruster Layout -->
     <xacro:include filename="${thruster_layout}"/>

Commit message: Feat: Change wamv to new mesh

File: wamv_description/urdf/wamv_base_contact.urdf.xacro (robot description, xacro)
@@ -112,6 +112,9 @@
     <visual>
       <geometry>
-        <mesh filename="package://wamv_description/models/WAM-V-Base/mesh/WAM-V-Base.dae"/>
+        <mesh filename="package://wamv_description/models/WAM-V-Base/mesh/WAM-V-Base.stl"/>
       </geometry>
+      <material name="wamv_visual_material">
+        <color rgba=".175 .175 .175  1.0" />
+      </material>
     </visual>
     <!-- Left base collisions -->
@@ -132,3 +135,6 @@
     </inertial>
   </link>
+  <gazebo reference="${namespace}/dummy_link">
+    <material>Gazebo/DarkGrey</material>
+  </gazebo>
 </robot>
